File: CAD/ECAD/_saved_ECAD.sch (KiCad schematic (older format))
At the start: 11 parts

Commit message: added Sound code
Parts:
- R? (x4): value 50KR -> 1KR
Connections:
- net labels added: +3.3V
- wire segments 35 -> 36
Changed lines of the file:
@@
 P 6750 4200
 F 0 "R?" H 6820 4246 50  0000 L CNN
-F 1 "50KR" H 6820 4155 50  0000 L CNN
+F 1 "1KR" H 6820 4155 50  0000 L CNN
 F 2 "" V 6680 4200 50  0001 C CNN
 F 3 "~" H 6750 4200 50  0001 C CNN
@@
 P 6900 4050
 F 0 "R?" V 7107 4050 50  0000 C CNN
-F 1 "50KR" V 7016 4050 50  0000 C CNN
+F 1 "1KR" V 7016 4050 50  0000 C CNN
 F 2 "" V 6830 4050 50  0001 C CNN
 F 3 "~" H 6900 4050 50  0001 C CNN
@@
 P 6750 3650
 F 0 "R?" H 6820 3696 50  0000 L CNN
-F 1 "50KR" H 6820 3605 50  0000 L CNN
+F 1 "1KR" H 6820 3605 50  0000 L CNN
 F 2 "" V 6680 3650 50  0001 C CNN
 F 3 "~" H 6750 3650 50  0001 C CNN
@@
 P 6900 3500
 F 0 "R?" V 7107 3500 50  0000 C CNN
-F 1 "50KR" V 7016 3500 50  0000 C CNN
+F 1 "1KR" V 7016 3500 50  0000 C CNN
 F 2 "" V 6830 3500 50  0001 C CNN
 F 3 "~" H 6900 3500 50  0001 C CNN
@@
 Wire Wire Line
 	6050 3500 6050 4450
-Wire Wire Line
-	6050 4450 5350 4450
-Wire Wire Line
-	5350 4450 5350 4350
 Connection ~ 6750 3500
 $Comp
@@
 Wire Wire Line
 	6750 4050 5900 4050
-Wire Wire Line
-	5900 4050 5900 4350
-Wire Wire Line
-	5900 4350 5450 4350
 Connection ~ 6750 4050
 Wire Wire Line
@@
 Wire Wire Line
 	7150 3600 7900 3600
+Wire Wire Line
+	5900 4400 5350 4400
+Wire Wire Line
+	5350 4400 5350 4350
+Wire Wire Line
+	5900 4050 5900 4400
+Wire Wire Line
+	5250 4450 5250 4350
+Wire Wire Line
+	5250 4450 6050 4450
+$Comp
+L power:+3.3V #PWR?
+U 1 1 5C9034DF
+P 8400 2800
+F 0 "#PWR?" H 8400 2650 50  0001 C CNN
+F 1 "+3.3V" H 8415 2973 50  0000 C CNN
+F 2 "" H 8400 2800 50  0001 C CNN
+F 3 "" H 8400 2800 50  0001 C CNN
+	1    8400 2800
+	1    0    0    -1
+$EndComp
+$Comp
+L power:GND #PWR?
+U 1 1 5C90358C
+P 8400 5000
+F 0 "#PWR?" H 8400 4750 50  0001 C CNN
+F 1 "GND" H 8405 4827 50  0000 C CNN
+F 2 "" H 8400 5000 50  0001 C CNN
+F 3 "" H 8400 5000 50  0001 C CNN
+	1    8400 5000
+	1    0    0    -1
+$EndComp
 $EndSCHEMATC
